File: hotdoggu_slimeVR_PCB.kicad_pcb (KiCad board)
At the start: 2 copper layers, 18.8 x 88.6 mm, 8 parts, among them J1 Conn_01x04_Pin, J2 Conn_01x02_Pin, SW1 SW_SPDT_312, U2 module_mpu6050

Commit message: some line changes
Routing:
- net +BATT: track 12.5 -> 13.5 mm
- net /VBAT_SW: track 58.8 -> 58.7 mm, vias 2 -> 1
Changed lines of the file:
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@@
 	)
 	(segment
-		(start 157.41 127)
-		(end 158 126.41)
+		(start 150.25 116.25)
+		(end 150.25 89.772)
+		(width 0.2)
+		(layer "F.Cu")
+		(net 2)
+	)
+	(segment
+		(start 157.5 126.91)
+		(end 157.5 123.5)
 		(width 0.2)
 		(layer "F.Cu")
@@
 	)
 	(segment
-		(start 150.25 101.5)
-		(end 150.25 95.272)
-		(width 0.2)
-		(layer "F.Cu")
-		(net 2)
-	)
-	(segment
 		(start 146.5 57.26)
 		(end 149.208 57.26)
@@
 	)
 	(segment
+		(start 157.41 127)
+		(end 157.5 126.91)
+		(width 0.2)
+		(layer "F.Cu")
+		(net 2)
+	)
+	(segment
+		(start 157.5 123.5)
+		(end 150.25 116.25)
+		(width 0.2)
+		(layer "F.Cu")
+		(net 2)
+	)
+	(segment
 		(start 150.25 82.749998)
 		(end 150.25 89.772)
@@
 	(segment
 		(start 150.25 89.772)
-		(end 150.25 95.272)
-		(width 0.2)
-		(layer "F.Cu")
-		(net 2)
-	)
-	(segment
-		(start 158 126.41)
-		(end 158 109.25)
-		(width 0.2)
-		(layer "F.Cu")
-		(net 2)
-	)
-	(segment
-		(start 158 109.25)
-		(end 150.25 101.5)
-		(width 0.2)
-		(layer "F.Cu")
-		(net 2)
-	)
-	(segment
-		(start 150.25 89.772)
 		(end 147.5 92.522)
 		(width 0.2)
@@
 	)
 	(segment
-		(start 156.22 112.543)
+		(start 148.108 121.666)
 		(end 148.108 120.655)
 		(width 0.4)
-		(layer "F.Cu")
+		(layer "B.Cu")
 		(net 17)
 	)
 	(segment
-		(start 157.25 106)
-		(end 161 106)
-		(width 0.4)
-		(layer "F.Cu")
-		(net 24)
+		(start 148.108 120.655)
+		(end 156.22 112.543)
+		(width 0.4)
+		(layer "B.Cu")
+		(net 17)
 	)
 	(segment
@@
 	)
 	(segment
+		(start 157.5 106)
+		(end 161 106)
+		(width 0.4)
+		(layer "F.Cu")
+		(net 24)
+	)
+	(segment
+		(start 150.46 74.645)
+		(end 150.46 71.71)
+		(width 0.4)
+		(layer "F.Cu")
+		(net 24)
+	)
+	(segment
 		(start 162.11 107.11)
 		(end 162.11 108.94)
@@
 	)
 	(segment
-		(start 150.46 74.645)
-		(end 150.46 71.71)
+		(start 156.22 107.28)
+		(end 157.5 106)
+		(width 0.4)
+		(layer "F.Cu")
+		(net 24)
+	)
+	(segment
+		(start 156.22 110.043)
+		(end 156.22 107.28)
 		(width 0.4)
 		(layer "F.Cu")
@@
 		(net 24)
 	)
-	(via
-		(at 157.25 106)
-		(size 0.6)
-		(drill 0.3)
-		(layers "F.Cu" "B.Cu")
-		(net 24)
-	)
 	(segment
 		(start 162.11 108.79858)
@@
 	)
 	(segment
-		(start 156.22 107.03)
-		(end 157.25 106)
-		(width 0.4)
-		(layer "B.Cu")
-		(net 24)
-	)
-	(segment
 		(start 150.75 88.5)
 		(end 150.75 74.935)
 		(width 0.4)
 		(layer "B.Cu")
-		(net 24)
-	)
-	(segment
-		(start 156.22 110.043)
-		(end 156.22 107.03)
-		(width 0.4)
-		(layer "B.Cu")
